File: kicad/v1/AtomRamAndNoiseKiller.sch (KiCad schematic (older format))
At the start: 21 parts, among them J1 Conn_02x10_Counter_Clockwise, J2 Conn_01x02, J3 Conn_01x02, J4 Conn_01x09, J5 Conn_01x09, J6 Conn_01x03, U1 74LS123, U2 74LS00, U3 74LS245, U4 74LS573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

Commit message: KiCad: Fully routed
Parts:
- removed J1: Conn_02x10_Counter_Clockwise, Package_DIP:DIP-20_W7.62mm_Socket, symbol Connector_Generic:Conn_02x10_Counter_Clockwise
- removed J2: Conn_01x02, Connector_PinHeader_2.54mm:PinHeader_1x02_P2.54mm_Vertical, symbol Connector_Generic:Conn_01x02
- removed U5: 8Kx8 SRAM, Package_DIP:DIP-28_W15.24mm_Socket, symbol Memory_NVRAM:FM1608B-SG
- added J1, J2: Conn_01x10, footprints:FinePinHeader_1x10_P2.54mm_Vertical, symbol Connector_Generic:Conn_01x10
- added J7: Conn_01x01, Connector_PinHeader_2.54mm:PinHeader_1x01_P2.54mm_Horizontal, symbol Connector_Generic:Conn_01x01
- added U5: 8Kx8 SRAM, Package_DIP:DIP-28_W15.24mm_Socket, symbol local:Generic_32Kx8_SRAM
- C1, C2, C3, C4, C5: footprint Capacitor_THT:C_Rect_L7.0mm_W2.0mm_P5.00mm -> Capacitor_THT:C_Axial_L3.8mm_D2.6mm_P7.50mm_Horizontal
- J4, J5: footprint Connector_PinHeader_2.54mm:PinHeader_1x09_P2.54mm_Vertical -> footprints:FinePinHeader_1x09_P2.54mm_Vertical
- J6: footprint Connector_PinHeader_2.54mm:PinHeader_1x03_P2.54mm_Vertical -> footprints:FinePinHeader_1x03_P2.54mm_Vertical
Connections:
- net A0: now also U5.8 (A2)
- net A1: now also U5.9 (A1)
- net A10: now also U5.2 (A12)
- net A11: now also U5.3 (A7)
- net A12: now also U5.4 (A6)
- net A2: now also U5.10 (A0)
- net A3: now also U5.7 (A3)
- net A4: now also U5.6 (A4)
- net A5: now also U5.5 (A5)
- net A6: now also U5.21 (A10)
- net A7: now also U5.25 (A8)
- net A8: now also U5.24 (A9)
- net A9: now also U5.23 (A11)
- net GND: now also J2.10 (Pin_10), U5.1 (A14), U5.14 (VSS), U5.20 (~CE~), U5.22 (~OE~), U5.26 (A13)
- net NDRS: now also J2.9 (Pin_9)
- net NVDG: now also J1.10 (Pin_10)
- net NWE: now also U5.27 (~WE~)
- net PD0: now also J2.1 (Pin_1)
- net PD1: now also J2.2 (Pin_2)
- net PD2: now also J2.3 (Pin_3)
- net PD3: now also J2.4 (Pin_4)
- net PD4: now also J2.5 (Pin_5)
- net PD5: now also J2.6 (Pin_6)
- net PD6: now also J2.7 (Pin_7)
- net PD7: now also J2.8 (Pin_8)
- net RD0: now also U5.19 (DQ7)
- net RD1: now also U5.18 (DQ6)
- net RD2: now also U5.17 (DQ5)
- net RD3: now also U5.16 (DQ4)
- net RD4: now also U5.15 (DQ3)
- net RD5: now also U5.11 (DQ0)
- net RD6: now also U5.12 (DQ1)
- net RD7: now also U5.13 (DQ2)
- net RRDISABLE: now also J7.1 (Pin_1)
- net VCC: now also J1.1 (Pin_1), U5.28 (VDD)
- net VD0: now also J1.2 (Pin_2)
- net VD1: now also J1.3 (Pin_3)
- net VD2: now also J1.4 (Pin_4)
- net VD3: now also J1.5 (Pin_5)
- net VD4: now also J1.6 (Pin_6)
- net VD5: now also J1.7 (Pin_7)
- net VD6: now also J1.8 (Pin_8)
- net VD7: now also J1.9 (Pin_9)
Changed lines of the file:
@@
-$EndComp
-$Comp
-L Connector_Generic:Conn_02x10_Counter_Clockwise J1
-U 1 1 5CB3180C
-P 1500 1750
-F 0 "J1" H 1550 2367 50  0000 C CNN
-F 1 "Conn_02x10_Counter_Clockwise" H 1550 2276 50  0000 C CNN
-F 2 "Package_DIP:DIP-20_W7.62mm_Socket" H 1500 1750 50  0001 C CNN
-F 3 "~" H 1500 1750 50  0001 C CNN
-	1    1500 1750
-	1    0    0    -1
 $EndComp
 $Comp
@@
 F 0 "J6" H 6900 4400 50  0000 L CNN
 F 1 "Conn_01x03" H 6850 4300 50  0000 L CNN
-F 2 "Connector_PinHeader_2.54mm:PinHeader_1x03_P2.54mm_Vertical" H 6950 4100 50  0001 C CNN
+F 2 "footprints:FinePinHeader_1x03_P2.54mm_Vertical" H 6950 4100 50  0001 C CNN
 F 3 "~" H 6950 4100 50  0001 C CNN
 	1    6950 4100
@@
 F 0 "J4" H 6900 2400 50  0000 L CNN
 F 1 "Conn_01x09" H 6750 2300 50  0000 L CNN
-F 2 "Connector_PinHeader_2.54mm:PinHeader_1x09_P2.54mm_Vertical" H 6950 1800 50  0001 C CNN
+F 2 "footprints:FinePinHeader_1x09_P2.54mm_Vertical" H 6950 1800 50  0001 C CNN
 F 3 "~" H 6950 1800 50  0001 C CNN
 	1    6950 1800
@@
 F 0 "J5" H 6900 3650 50  0000 L CNN
 F 1 "Conn_01x09" H 6800 3550 50  0000 L CNN
-F 2 "Connector_PinHeader_2.54mm:PinHeader_1x09_P2.54mm_Vertical" H 6950 3050 50  0001 C CNN
+F 2 "footprints:FinePinHeader_1x09_P2.54mm_Vertical" H 6950 3050 50  0001 C CNN
 F 3 "~" H 6950 3050 50  0001 C CNN
 	1    6950 3050
@@
 F 0 "C1" H 4065 6996 50  0000 L CNN
 F 1 "100n" H 4065 6905 50  0000 L CNN
-F 2 "Capacitor_THT:C_Rect_L7.0mm_W2.0mm_P5.00mm" H 3988 6800 50  0001 C CNN
+F 2 "Capacitor_THT:C_Axial_L3.8mm_D2.6mm_P7.50mm_Horizontal" H 3988 6800 50  0001 C CNN
 F 3 "~" H 3950 6950 50  0001 C CNN
 	1    3950 6950
@@
 F 0 "C2" H 4515 6996 50  0000 L CNN
 F 1 "100n" H 4515 6905 50  0000 L CNN
-F 2 "Capacitor_THT:C_Rect_L7.0mm_W2.0mm_P5.00mm" H 4438 6800 50  0001 C CNN
+F 2 "Capacitor_THT:C_Axial_L3.8mm_D2.6mm_P7.50mm_Horizontal" H 4438 6800 50  0001 C CNN
 F 3 "~" H 4400 6950 50  0001 C CNN
 	1    4400 6950
@@
 F 0 "C3" H 4965 6996 50  0000 L CNN
 F 1 "100n" H 4965 6905 50  0000 L CNN
-F 2 "Capacitor_THT:C_Rect_L7.0mm_W2.0mm_P5.00mm" H 4888 6800 50  0001 C CNN
+F 2 "Capacitor_THT:C_Axial_L3.8mm_D2.6mm_P7.50mm_Horizontal" H 4888 6800 50  0001 C CNN
 F 3 "~" H 4850 6950 50  0001 C CNN
 	1    4850 6950
@@
 F 0 "C4" H 5415 6996 50  0000 L CNN
 F 1 "100n" H 5415 6905 50  0000 L CNN
-F 2 "Capacitor_THT:C_Rect_L7.0mm_W2.0mm_P5.00mm" H 5338 6800 50  0001 C CNN
+F 2 "Capacitor_THT:C_Axial_L3.8mm_D2.6mm_P7.50mm_Horizontal" H 5338 6800 50  0001 C CNN
 F 3 "~" H 5300 6950 50  0001 C CNN
 	1    5300 6950
@@
 F 0 "C5" H 5815 6996 50  0000 L CNN
 F 1 "100n" H 5815 6905 50  0000 L CNN
-F 2 "Capacitor_THT:C_Rect_L7.0mm_W2.0mm_P5.00mm" H 5738 6800 50  0001 C CNN
+F 2 "Capacitor_THT:C_Axial_L3.8mm_D2.6mm_P7.50mm_Horizontal" H 5738 6800 50  0001 C CNN
 F 3 "~" H 5700 6950 50  0001 C CNN
 	1    5700 6950
@@
 Wire Wire Line
 	1800 2050 2350 2050
-Text Label 1300 1350 2    50   ~ 0
+Text Label 1200 1350 2    50   ~ 0
 VCC
 Text Label 1800 2250 0    50   ~ 0
@@
 L power:GND #PWR013
 U 1 1 5CB33943
-P 8250 2850
-F 0 "#PWR013" H 8250 2600 50  0001 C CNN
-F 1 "GND" H 8255 2677 50  0000 C CNN
-F 2 "" H 8250 2850 50  0001 C CNN
-F 3 "" H 8250 2850 50  0001 C CNN
-	1    8250 2850
-	1    0    0    -1
-$EndComp
-Text Label 7750 1450 2    50   ~ 0
+P 8250 3050
+F 0 "#PWR013" H 8250 2800 50  0001 C CNN
+F 1 "GND" H 8255 2877 50  0000 C CNN
+F 2 "" H 8250 3050 50  0001 C CNN
+F 3 "" H 8250 3050 50  0001 C CNN
+	1    8250 3050
+	1    0    0    -1
+$EndComp
+Text Label 7750 1650 2    50   ~ 0
 A0
 Text Label 7750 1550 2    50   ~ 0
 A1
-Text Label 7750 1650 2    50   ~ 0
+Text Label 7750 1450 2    50   ~ 0
 A2
 Text Label 7750 1750 2    50   ~ 0
@@
 Text Label 7750 1950 2    50   ~ 0
 A5
+Text Label 7750 2450 2    50   ~ 0
+A6
+Text Label 7750 2250 2    50   ~ 0
+A7
+Text Label 7750 2350 2    50   ~ 0
+A8
+Text Label 7750 2550 2    50   ~ 0
+A9
+Text Label 7750 2650 2    50   ~ 0
+A10
+Text Label 7750 2150 2    50   ~ 0
+A11
 Text Label 7750 2050 2    50   ~ 0
-A6
-Text Label 7750 2150 2    50   ~ 0
-A7
-Text Label 7750 2250 2    50   ~ 0
-A8
-Text Label 7750 2350 2    50   ~ 0
-A9
-Text Label 7750 2450 2    50   ~ 0
-A10
-Text Label 7750 2550 2    50   ~ 0
-A11
-Text Label 7750 2650 2    50   ~ 0
 A12
-Text Label 8750 2350 0    50   ~ 0
+Text Label 8750 2550 0    50   ~ 0
+GND
+Text Label 8750 2850 0    50   ~ 0
 GND
 Text Label 8750 2650 0    50   ~ 0
-GND
-Text Label 8750 2450 0    50   ~ 0
 NWE
+Text Label 8750 2150 0    50   ~ 0
+RD0
+Text Label 8750 2050 0    50   ~ 0
+RD1
+Text Label 8750 1950 0    50   ~ 0
+RD2
+Text Label 8750 1850 0    50   ~ 0
+RD3
+Text Label 8750 1750 0    50   ~ 0
+RD4
 Text Label 8750 1450 0    50   ~ 0
-RD0
+RD5
 Text Label 8750 1550 0    50   ~ 0
-RD1
+RD6
 Text Label 8750 1650 0    50   ~ 0
-RD2
-Text Label 8750 1750 0    50   ~ 0
-RD3
-Text Label 8750 1850 0    50   ~ 0
-RD4
-Text Label 8750 1950 0    50   ~ 0
-RD5
-Text Label 8750 2050 0    50   ~ 0
-RD6
-Text Label 8750 2150 0    50   ~ 0
 RD7
 $Comp
@@
 Text Label 6750 4200 2    50   ~ 0
 A12
-$Comp
-L Memory_NVRAM:FM1608B-SG U5
-U 1 1 5CB3EB15
-P 8250 2050
-F 0 "U5" H 7750 2900 50  0000 C CNN
-F 1 "8Kx8 SRAM" H 7850 2800 50  0000 C CNN
-F 2 "Package_DIP:DIP-28_W15.24mm_Socket" H 8250 2050 50  0001 C CNN
-F 3 "http://www.cypress.com/file/41731/download" H 8250 2050 50  0001 C CNN
-	1    8250 2050
-	1    0    0    -1
-$EndComp
 Wire Wire Line
 	2300 3900 2750 3900
@@
 Text Label 5850 4600 0    50   ~ 0
 LOAD
-$Comp
-L Connector_Generic:Conn_01x02 J2
-U 1 1 5CB4D0F5
-P 3000 5000
-F 0 "J2" H 2920 4675 50  0000 C CNN
-F 1 "Conn_01x02" H 2920 4766 50  0000 C CNN
-F 2 "Connector_PinHeader_2.54mm:PinHeader_1x02_P2.54mm_Vertical" H 3000 5000 50  0001 C CNN
-F 3 "~" H 3000 5000 50  0001 C CNN
-	1    3000 5000
-	-1   0    0    1
-$EndComp
 Wire Wire Line
 	4200 4800 4000 4800
@@
 Wire Wire Line
 	4000 4900 4000 5000
-Wire Wire Line
-	3200 5000 3300 5000
-Wire Wire Line
-	3300 5000 3300 4900
-Wire Wire Line
-	3300 4900 3200 4900
-Wire Wire Line
-	3300 4900 3450 4900
-Connection ~ 3300 4900
 Connection ~ 3450 4900
 Text Label 3450 4900 0    50   ~ 0
@@
 	2350 2150 1800 2150
 Wire Wire Line
-	1300 2250 1300 2350
-Wire Wire Line
-	1300 2350 2350 2350
-Text Label 1300 1450 2    50   ~ 0
+	1200 2250 1200 2350
+Wire Wire Line
+	1200 2350 2350 2350
+Text Label 1200 1450 2    50   ~ 0
 VD0
-Text Label 1300 1550 2    50   ~ 0
+Text Label 1200 1550 2    50   ~ 0
 VD1
-Text Label 1300 1650 2    50   ~ 0
+Text Label 1200 1650 2    50   ~ 0
 VD2
-Text Label 1300 1750 2    50   ~ 0
+Text Label 1200 1750 2    50   ~ 0
 VD3
-Text Label 1300 1850 2    50   ~ 0
+Text Label 1200 1850 2    50   ~ 0
 VD4
-Text Label 1300 1950 2    50   ~ 0
+Text Label 1200 1950 2    50   ~ 0
 VD5
-Text Label 1300 2050 2    50   ~ 0
+Text Label 1200 2050 2    50   ~ 0
 VD6
-Text Label 1300 2150 2    50   ~ 0
+Text Label 1200 2150 2    50   ~ 0
 VD7
+$Comp
+L Connector_Generic:Conn_01x10 J2
+U 1 1 5CB35F97
+P 1600 1750
+F 0 "J2" H 1600 2400 50  0000 C CNN
+F 1 "Conn_01x10" H 1450 2300 50  0000 C CNN
+F 2 "footprints:FinePinHeader_1x10_P2.54mm_Vertical" H 1600 1750 50  0001 C CNN
+F 3 "~" H 1600 1750 50  0001 C CNN
+	1    1600 1750
+	-1   0    0    -1
+$EndComp
+$Comp
+L Connector_Generic:Conn_01x10 J1
+U 1 1 5CB360B1
+P 1400 1750
+F 0 "J1" H 1350 2400 50  0000 L CNN
+F 1 "Conn_01x10" H 1000 2300 50  0000 L CNN
+F 2 "footprints:FinePinHeader_1x10_P2.54mm_Vertical" H 1400 1750 50  0001 C CNN
+F 3 "~" H 1400 1750 50  0001 C CNN
+	1    1400 1750
+	1    0    0    -1
+$EndComp
+$Comp
+L Connector_Generic:Conn_01x01 J7
+U 1 1 5CB4564A
+P 3000 4900
+F 0 "J7" H 2920 4675 50  0000 C CNN
+F 1 "Conn_01x01" H 2920 4766 50  0000 C CNN
+F 2 "Connector_PinHeader_2.54mm:PinHeader_1x01_P2.54mm_Horizontal" H 3000 4900 50  0001 C CNN
+F 3 "~" H 3000 4900 50  0001 C CNN
+	1    3000 4900
+	-1   0    0    1
+$EndComp
+Wire Wire Line
+	3200 4900 3450 4900
+$Comp
+L local:Generic_32Kx8_SRAM U5
+U 1 1 5CB46E17
+P 8250 2150
+F 0 "U5" H 7900 3100 50  0000 C CNN
+F 1 "8Kx8 SRAM" H 7900 3000 50  0000 C CNN
+F 2 "Package_DIP:DIP-28_W15.24mm_Socket" H 8250 2150 50  0001 C CNN
+F 3 "" H 8250 2250 50  0001 C CNN
+	1    8250 2150
+	1    0    0    -1
+$EndComp
+Text Label 7750 2850 2    50   ~ 0
+GND
+Text Label 7750 2750 2    50   ~ 0
+GND
 $EndSCHEMATC

Commit message: More work
Parts:
- added J3: Conn_01x03, footprints:FinePinHeader_1x03_P2.54mm_Vertical, symbol Connector_Generic:Conn_01x03
- renumbered J3 to J7, J7 to J8
Connections:
- net NWE: now also J3.3 (Pin_3); no longer J5.9 (Pin_9)
- no-connect marks 10 -> 13
Other:
- moved on the sheet: J4, J5, J6, U5
Changed lines of the file:
@@
 L Connector_Generic:Conn_01x03 J6
 U 1 1 5CB31891
-P 6950 4100
-F 0 "J6" H 6900 4400 50  0000 L CNN
-F 1 "Conn_01x03" H 6850 4300 50  0000 L CNN
-F 2 "footprints:FinePinHeader_1x03_P2.54mm_Vertical" H 6950 4100 50  0001 C CNN
-F 3 "~" H 6950 4100 50  0001 C CNN
-	1    6950 4100
+P 8050 4700
+F 0 "J6" H 8000 5000 50  0000 L CNN
+F 1 "Conn_01x03" H 7950 4900 50  0000 L CNN
+F 2 "footprints:FinePinHeader_1x03_P2.54mm_Vertical" H 8050 4700 50  0001 C CNN
+F 3 "~" H 8050 4700 50  0001 C CNN
+	1    8050 4700
 	1    0    0    -1
 $EndComp
@@
 L Connector_Generic:Conn_01x09 J4
 U 1 1 5CB3198E
-P 6950 1800
-F 0 "J4" H 6900 2400 50  0000 L CNN
-F 1 "Conn_01x09" H 6750 2300 50  0000 L CNN
-F 2 "footprints:FinePinHeader_1x09_P2.54mm_Vertical" H 6950 1800 50  0001 C CNN
-F 3 "~" H 6950 1800 50  0001 C CNN
-	1    6950 1800
+P 8050 2400
+F 0 "J4" H 8000 3000 50  0000 L CNN
+F 1 "Conn_01x09" H 7850 2900 50  0000 L CNN
+F 2 "footprints:FinePinHeader_1x09_P2.54mm_Vertical" H 8050 2400 50  0001 C CNN
+F 3 "~" H 8050 2400 50  0001 C CNN
+	1    8050 2400
 	1    0    0    -1
 $EndComp
@@
 L Connector_Generic:Conn_01x09 J5
 U 1 1 5CB319E9
-P 6950 3050
-F 0 "J5" H 6900 3650 50  0000 L CNN
-F 1 "Conn_01x09" H 6800 3550 50  0000 L CNN
-F 2 "footprints:FinePinHeader_1x09_P2.54mm_Vertical" H 6950 3050 50  0001 C CNN
-F 3 "~" H 6950 3050 50  0001 C CNN
-	1    6950 3050
+P 8050 3650
+F 0 "J5" H 8000 4250 50  0000 L CNN
+F 1 "Conn_01x09" H 7900 4150 50  0000 L CNN
+F 2 "footprints:FinePinHeader_1x09_P2.54mm_Vertical" H 8050 3650 50  0001 C CNN
+F 3 "~" H 8050 3650 50  0001 C CNN
+	1    8050 3650
 	1    0    0    -1
 $EndComp
@@
 L power:VCC #PWR012
 U 1 1 5CB33914
-P 8250 1250
-F 0 "#PWR012" H 8250 1100 50  0001 C CNN
-F 1 "VCC" H 8267 1423 50  0000 C CNN
-F 2 "" H 8250 1250 50  0001 C CNN
-F 3 "" H 8250 1250 50  0001 C CNN
-	1    8250 1250
-	1    0    0    -1
+P 6050 1100
+F 0 "#PWR012" H 6050 950 50  0001 C CNN
+F 1 "VCC" H 6067 1273 50  0000 C CNN
+F 2 "" H 6050 1100 50  0001 C CNN
+F 3 "" H 6050 1100 50  0001 C CNN
+	1    6050 1100
+	-1   0    0    -1
 $EndComp
 $Comp
 L power:GND #PWR013
 U 1 1 5CB33943
-P 8250 3050
-F 0 "#PWR013" H 8250 2800 50  0001 C CNN
-F 1 "GND" H 8255 2877 50  0000 C CNN
-F 2 "" H 8250 3050 50  0001 C CNN
-F 3 "" H 8250 3050 50  0001 C CNN
-	1    8250 3050
-	1    0    0    -1
-$EndComp
-Text Label 7750 1650 2    50   ~ 0
+P 6050 2900
+F 0 "#PWR013" H 6050 2650 50  0001 C CNN
+F 1 "GND" H 6055 2727 50  0000 C CNN
+F 2 "" H 6050 2900 50  0001 C CNN
+F 3 "" H 6050 2900 50  0001 C CNN
+	1    6050 2900
+	-1   0    0    -1
+$EndComp
+Text Label 6550 1500 0    50   ~ 0
 A0
-Text Label 7750 1550 2    50   ~ 0
+Text Label 6550 1400 0    50   ~ 0
 A1
-Text Label 7750 1450 2    50   ~ 0
+Text Label 6550 1300 0    50   ~ 0
 A2
-Text Label 7750 1750 2    50   ~ 0
+Text Label 6550 1600 0    50   ~ 0
 A3
-Text Label 7750 1850 2    50   ~ 0
+Text Label 6550 1700 0    50   ~ 0
 A4
-Text Label 7750 1950 2    50   ~ 0
+Text Label 6550 1800 0    50   ~ 0
 A5
-Text Label 7750 2450 2    50   ~ 0
+Text Label 6550 2300 0    50   ~ 0
 A6
-Text Label 7750 2250 2    50   ~ 0
+Text Label 6550 2100 0    50   ~ 0
 A7
-Text Label 7750 2350 2    50   ~ 0
+Text Label 6550 2200 0    50   ~ 0
 A8
-Text Label 7750 2550 2    50   ~ 0
+Text Label 6550 2400 0    50   ~ 0
 A9
-Text Label 7750 2650 2    50   ~ 0
+Text Label 6550 2500 0    50   ~ 0
 A10
-Text Label 7750 2150 2    50   ~ 0
+Text Label 6550 2000 0    50   ~ 0
 A11
-Text Label 7750 2050 2    50   ~ 0
+Text Label 6550 1900 0    50   ~ 0
 A12
-Text Label 8750 2550 0    50   ~ 0
+Text Label 5550 2400 2    50   ~ 0
 GND
-Text Label 8750 2850 0    50   ~ 0
+Text Label 5550 2700 2    50   ~ 0
 GND
-Text Label 8750 2650 0    50   ~ 0
+Text Label 5550 2500 2    50   ~ 0
 NWE
-Text Label 8750 2150 0    50   ~ 0
+Text Label 5550 2000 2    50   ~ 0
 RD0
-Text Label 8750 2050 0    50   ~ 0
+Text Label 5550 1900 2    50   ~ 0
 RD1
-Text Label 8750 1950 0    50   ~ 0
+Text Label 5550 1800 2    50   ~ 0
 RD2
-Text Label 8750 1850 0    50   ~ 0
+Text Label 5550 1700 2    50   ~ 0
 RD3
-Text Label 8750 1750 0    50   ~ 0
+Text Label 5550 1600 2    50   ~ 0
 RD4
-Text Label 8750 1450 0    50   ~ 0
+Text Label 5550 1300 2    50   ~ 0
 RD5
-Text Label 8750 1550 0    50   ~ 0
+Text Label 5550 1400 2    50   ~ 0
 RD6
-Text Label 8750 1650 0    50   ~ 0
+Text Label 5550 1500 2    50   ~ 0
 RD7
 $Comp
@@
 	1    0    0    -1
 $EndComp
-Text Label 6750 3450 2    50   ~ 0
+Text Label 7850 1500 2    50   ~ 0
 NWE
-NoConn ~ 6750 2100
-NoConn ~ 6750 3050
-NoConn ~ 6750 3150
-NoConn ~ 6750 3250
-NoConn ~ 6750 3350
-Text Label 6750 1400 2    50   ~ 0
+NoConn ~ 7850 2700
+NoConn ~ 7850 3650
+NoConn ~ 7850 3750
+NoConn ~ 7850 3850
+NoConn ~ 7850 3950
+Text Label 7850 2000 2    50   ~ 0
 A6
-Text Label 6750 1500 2    50   ~ 0
+Text Label 7850 2100 2    50   ~ 0
 A5
-Text Label 6750 1600 2    50   ~ 0
+Text Label 7850 2200 2    50   ~ 0
 A4
-Text Label 6750 1700 2    50   ~ 0
+Text Label 7850 2300 2    50   ~ 0
 A3
-Text Label 6750 1800 2    50   ~ 0
+Text Label 7850 2400 2    50   ~ 0
 A0
-Text Label 6750 1900 2    50   ~ 0
+Text Label 7850 2500 2    50   ~ 0
 A1
-Text Label 6750 2000 2    50   ~ 0
+Text Label 7850 2600 2    50   ~ 0
 A2
-Text Label 6750 2200 2    50   ~ 0
+Text Label 7850 2800 2    50   ~ 0
 GND
-Text Label 6750 2650 2    50   ~ 0
+Text Label 7850 3250 2    50   ~ 0
 VCC
-Text Label 6750 2750 2    50   ~ 0
+Text Label 7850 3350 2    50   ~ 0
 A7
-Text Label 6750 2850 2    50   ~ 0
+Text Label 7850 3450 2    50   ~ 0
 A8
-Text Label 6750 2950 2    50   ~ 0
+Text Label 7850 3550 2    50   ~ 0
 A9
-Text Label 6750 4000 2    50   ~ 0
+Text Label 7850 4600 2    50   ~ 0
 A10
-Text Label 6750 4100 2    50   ~ 0
+Text Label 7850 4700 2    50   ~ 0
 A11
-Text Label 6750 4200 2    50   ~ 0
+Text Label 7850 4800 2    50   ~ 0
 A12
 Wire Wire Line
@@
 LOAD
 $Comp
-L Connector_Generic:Conn_01x02 J3
+L Connector_Generic:Conn_01x02 J7
 U 1 1 5CB48B01
 P 5650 4800
-F 0 "J3" V 5523 4880 50  0000 L CNN
+F 0 "J7" V 5523 4880 50  0000 L CNN
 F 1 "Conn_01x02" V 5614 4880 50  0000 L CNN
 F 2 "Connector_PinHeader_2.54mm:PinHeader_1x02_P2.54mm_Vertical" H 5650 4800 50  0001 C CNN
@@
 	5650 4600 6100 4600
 Wire Wire Line
-	6100 4600 6100 2950
-Wire Wire Line
-	6100 2950 3600 2950
-Wire Wire Line
-	3600 2950 3600 2250
+	6100 4600 6100 3450
+Wire Wire Line
+	6100 3450 3600 3450
+Wire Wire Line
+	3600 3450 3600 2250
 Wire Wire Line
 	3600 2250 3950 2250
@@
 	1200 2250 1200 2350
 Wire Wire Line
-	1200 2350 2350 2350
-Text Label 1200 1450 2    50   ~ 0
-VD0
-Text Label 1200 1550 2    50   ~ 0
-VD1
-Text Label 1200 1650 2    50   ~ 0
-VD2
-Text Label 1200 1750 2    50   ~ 0
-VD3
-Text Label 1200 1850 2    50   ~ 0
-VD4
-Text Label 1200 1950 2    50   ~ 0
-VD5
-Text Label 1200 2050 2    50   ~ 0
-VD6
-Text Label 1200 2150 2    50   ~ 0
-VD7
+	1200 2350 2100 2350
 $Comp
 L Connector_Generic:Conn_01x10 J2
@@
 $EndComp
 $Comp
-L Connector_Generic:Conn_01x01 J7
+L Connector_Generic:Conn_01x01 J8
 U 1 1 5CB4564A
 P 3000 4900
-F 0 "J7" H 2920 4675 50  0000 C CNN
+F 0 "J8" H 2920 4675 50  0000 C CNN
 F 1 "Conn_01x01" H 2920 4766 50  0000 C CNN
 F 2 "Connector_PinHeader_2.54mm:PinHeader_1x01_P2.54mm_Horizontal" H 3000 4900 50  0001 C CNN
@@
 L local:Generic_32Kx8_SRAM U5
 U 1 1 5CB46E17
-P 8250 2150
-F 0 "U5" H 7900 3100 50  0000 C CNN
-F 1 "8Kx8 SRAM" H 7900 3000 50  0000 C CNN
-F 2 "Package_DIP:DIP-28_W15.24mm_Socket" H 8250 2150 50  0001 C CNN
-F 3 "" H 8250 2250 50  0001 C CNN
-	1    8250 2150
-	1    0    0    -1
-$EndComp
-Text Label 7750 2850 2    50   ~ 0
+P 6050 2000
+F 0 "U5" H 5700 2950 50  0000 C CNN
+F 1 "8Kx8 SRAM" H 5700 2850 50  0000 C CNN
+F 2 "Package_DIP:DIP-28_W15.24mm_Socket" H 6050 2000 50  0001 C CNN
+F 3 "" H 6050 2100 50  0001 C CNN
+	1    6050 2000
+	-1   0    0    -1
+$EndComp
+Text Label 6550 2700 0    50   ~ 0
 GND
-Text Label 7750 2750 2    50   ~ 0
+Text Label 6550 2600 0    50   ~ 0
 GND
+Wire Wire Line
+	2100 2350 2100 4100
+Wire Wire Line
+	2100 4100 2750 4100
+Connection ~ 2100 2350
+Wire Wire Line
+	2100 2350 2350 2350
+Wire Wire Line
+	4200 4400 3800 4400
+Wire Wire Line
+	3800 4400 3800 4600
+Wire Wire Line
+	3800 4600 2100 4600
+Wire Wire Line
+	2100 4600 2100 4100
+Connection ~ 2100 4100
+$Comp
+L Connector_Generic:Conn_01x03 J3
+U 1 1 5CB4E2B2
+P 8050 1400
+F 0 "J3" H 8000 1700 50  0000 L CNN
+F 1 "Conn_01x03" H 7950 1600 50  0000 L CNN
+F 2 "footprints:FinePinHeader_1x03_P2.54mm_Vertical" H 8050 1400 50  0001 C CNN
+F 3 "~" H 8050 1400 50  0001 C CNN
+	1    8050 1400
+	1    0    0    -1
+$EndComp
+NoConn ~ 7850 4050
+NoConn ~ 7850 1400
+NoConn ~ 7850 1300
+Text Label 1200 2150 2    50   ~ 0
+VD7
+Text Label 1200 2050 2    50   ~ 0
+VD6
+Text Label 1200 1950 2    50   ~ 0
+VD5
+Text Label 1200 1850 2    50   ~ 0
+VD4
+Text Label 1200 1750 2    50   ~ 0
+VD3
+Text Label 1200 1650 2    50   ~ 0
+VD2
+Text Label 1200 1550 2    50   ~ 0
+VD1
+Text Label 1200 1450 2    50   ~ 0
+VD0
 $EndSCHEMATC

Commit message: Almost finished
Parts:
- renumbered R3 to R2, R2 to R3
Changed lines of the file:
@@
 	5400 4600 5550 4600
 $Comp
-L Device:R R3
+L Device:R R2
 U 1 1 5CB49B94
 P 5650 4300
-F 0 "R3" H 5720 4346 50  0000 L CNN
+F 0 "R2" H 5720 4346 50  0000 L CNN
 F 1 "10K" H 5720 4255 50  0000 L CNN
 F 2 "Resistor_THT:R_Axial_DIN0207_L6.3mm_D2.5mm_P10.16mm_Horizontal" V 5580 4300 50  0001 C CNN
@@
 	4000 5000 4200 5000
 $Comp
-L Device:R R2
+L Device:R R3
 U 1 1 5CB4E6C0
 P 3450 5300
-F 0 "R2" H 3520 5346 50  0000 L CNN
+F 0 "R3" H 3520 5346 50  0000 L CNN
 F 1 "47K" H 3520 5255 50  0000 L CNN
 F 2 "Resistor_THT:R_Axial_DIN0207_L6.3mm_D2.5mm_P10.16mm_Horizontal" V 3380 5300 50  0001 C CNN
