File: kicad/v2/AtomRamAndNoiseKiller.sch (KiCad schematic (older format))
At the start: 27 parts, among them J1 Conn_01x10, J10 Conn_01x03, J2 Conn_01x10, J3 Conn_01x03, J4 Conn_01x09, J5 Conn_01x09, J6 Conn_01x03, J7 Conn_01x02, J8 Conn_01x01, J9 Conn_01x03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

Commit message: Final tweaks
Parts:
- renumbered J8 to J7, J10 to LK1, J9 to LK2, J7 to LK3
Changed lines of the file:
@@
 LOAD
 $Comp
-L Connector_Generic:Conn_01x02 J7
+L Connector_Generic:Conn_01x02 LK3
 U 1 1 5CB48B01
 P 5650 4800
-F 0 "J7" V 5523 4880 50  0000 L CNN
+F 0 "LK3" V 5523 4880 50  0000 L CNN
 F 1 "Conn_01x02" V 5614 4880 50  0000 L CNN
 F 2 "Connector_PinHeader_2.54mm:PinHeader_1x02_P2.54mm_Vertical" H 5650 4800 50  0001 C CNN
@@
 $EndComp
 $Comp
-L Connector_Generic:Conn_01x01 J8
+L Connector_Generic:Conn_01x01 J7
 U 1 1 5CB4564A
 P 3000 4900
-F 0 "J8" H 2920 4675 50  0000 C CNN
+F 0 "J7" H 2920 4675 50  0000 C CNN
 F 1 "Conn_01x01" H 2920 4766 50  0000 C CNN
 F 2 "Connector_PinHeader_2.54mm:PinHeader_1x01_P2.54mm_Horizontal" H 3000 4900 50  0001 C CNN
@@
 RAMNOE
 $Comp
-L Connector_Generic:Conn_01x03 J10
+L Connector_Generic:Conn_01x03 LK1
 U 1 1 5CD4E9A2
 P 5500 6550
-F 0 "J10" H 5580 6592 50  0000 L CNN
+F 0 "LK1" H 5580 6592 50  0000 L CNN
 F 1 "Conn_01x03" H 5580 6501 50  0000 L CNN
 F 2 "Connector_PinHeader_2.54mm:PinHeader_1x03_P2.54mm_Vertical" H 5500 6550 50  0001 C CNN
@@
 	5200 6650 5300 6650
 $Comp
-L Connector_Generic:Conn_01x03 J9
+L Connector_Generic:Conn_01x03 LK2
 U 1 1 5CD9FF58
 P 5500 5800
-F 0 "J9" H 5580 5842 50  0000 L CNN
+F 0 "LK2" H 5580 5842 50  0000 L CNN
 F 1 "Conn_01x03" H 5580 5751 50  0000 L CNN
 F 2 "Connector_PinHeader_2.54mm:PinHeader_1x03_P2.54mm_Vertical" H 5500 5800 50  0001 C CNN
